File: kicad/stepper_monitor.kicad_sch (KiCad schematic)
At the start: 57 parts, among them J1 Conn_01x04_Male, J2 Conn_01x04_Male, J3 Conn_01x02_Male, J4 USB_C_Receptacle_USB2.0, J5 JTAG, M1 Motor-simple_stepper_motor_an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, Q1 MMDT2222A, Q2 PJA3439, SW1 SW_Push, U1 CP2102N-A01-GQFN28, U2 AMS1117-3.3, U3 ESP32-WROOM-32U-N4, U4 5V, U5 CC6920BSO-5A, U6 CC6920BSO-5A

Commit message: Changed yellow LED to green.
Parts:
- D2: value YELLOW -> GREEN
- R5: LCSC C25905 -> C965797
Changed lines of the file:
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@@
       (effects (font (size 1.27 1.27)) (justify right))
     )
-    (property "Value" "YELLOW" (id 1) (at 43.815 177.165 90)
+    (property "Value" "GREEN" (id 1) (at 43.815 177.165 90)
       (effects (font (size 1.27 1.27)) (justify right))
     )
@@
       (effects (font (size 1.27 1.27)) hide)
     )
-    (property "LCSC" "C25905" (id 4) (at 36.195 170.815 0))
+    (property "LCSC" "C965797" (id 4) (at 36.195 170.815 0))
     (pin "1")
     (pin "2")
@@
     )
     (path "/00000000-0000-0000-0000-000063192ea5"
-      (reference "D2") (unit 1) (value "YELLOW") (footprint "stepper_monitor:LED_0402_1005Metric_Pad0.77x0.64mm_HandSolder")
+      (reference "D2") (unit 1) (value "GREEN") (footprint "stepper_monitor:LED_0402_1005Metric_Pad0.77x0.64mm_HandSolder")
     )
     (path "/00000000-0000-0000-0000-000063190058"

Commit message: Changed solder jumper to 0 ohms resistor.
Parts:
- removed JP1: SolderJumper_2_Open, stepper_monitor:SolderJumper-2_P1.3mm_Open_RoundedPad1.0x1.5mm, symbol Jumper:SolderJumper_2_Open
- added R19: 0R, Resistor_SMD:R_0402_1005Metric, symbol Device:R_Small_US
Connections:
- net +3V3: now also R19.1
- net at C3.2, C4.2, U2.2 (VO): now also R19.2
Other:
- note added: "ESP32 Stepper Motor Analyzer 1.4.1"
- note removed: "ESP32 Stepper Motor Analyzer 1.4.0"
Changed lines of the file:
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@@
   (junction (at 117.475 186.055) (diameter 0) (color 0 0 0 0)
   )
-  (junction (at 144.145 37.465) (diameter 0) (color 0 0 0 0)
+  (junction (at 145.415 37.465) (diameter 0) (color 0 0 0 0)
   )
   (junction (at 142.875 174.625) (diameter 0) (color 0 0 0 0)
@@
   (junction (at 103.505 69.85) (diameter 0) (color 0 0 0 0)
   )
+  (junction (at 93.98 51.435) (diameter 0) (color 0 0 0 0)
+  )
+  (junction (at 269.875 114.935) (diameter 0) (color 0 0 0 0)
+  )
+  (junction (at 117.475 160.655) (diameter 0) (color 0 0 0 0)
+  )
+  (junction (at 134.62 51.435) (diameter 0) (color 0 0 0 0)
+  )
+  (junction (at 214.63 26.67) (diameter 0) (color 0 0 0 0)
+  )
   (junction (at 134.62 37.465) (diameter 0) (color 0 0 0 0)
-  )
-  (junction (at 93.98 51.435) (diameter 0) (color 0 0 0 0)
-  )
-  (junction (at 269.875 114.935) (diameter 0) (color 0 0 0 0)
-  )
-  (junction (at 117.475 160.655) (diameter 0) (color 0 0 0 0)
-  )
-  (junction (at 134.62 51.435) (diameter 0) (color 0 0 0 0)
-  )
-  (junction (at 214.63 26.67) (diameter 0) (color 0 0 0 0)
   )
   (junction (at 91.44 179.705) (diameter 0) (color 0 0 0 0)
@@
     (stroke (width 0) (type default) (color 0 0 0 0))
   )
-  (wire (pts (xy 144.145 37.465) (xy 147.955 37.465))
+  (wire (pts (xy 145.415 37.465) (xy 149.225 37.465))
     (stroke (width 0) (type default) (color 0 0 0 0))
   )
@@
     (stroke (width 0) (type default) (color 0 0 0 0))
   )
+  (wire (pts (xy 134.62 37.465) (xy 137.16 37.465))
+    (stroke (width 0) (type default) (color 0 0 0 0))
+  )
   (wire (pts (xy 53.975 51.435) (xy 67.31 51.435))
     (stroke (width 0) (type default) (color 0 0 0 0))
@@
     (stroke (width 0) (type default) (color 0 0 0 0))
   )
-  (wire (pts (xy 144.145 36.83) (xy 144.145 37.465))
+  (wire (pts (xy 145.415 36.83) (xy 145.415 37.465))
     (stroke (width 0) (type default) (color 0 0 0 0))
   )
@@
     (stroke (width 0) (type default) (color 0 0 0 0))
   )
-  (wire (pts (xy 142.24 37.465) (xy 144.145 37.465))
+  (wire (pts (xy 142.24 37.465) (xy 145.415 37.465))
     (stroke (width 0) (type default) (color 0 0 0 0))
   )
@@
     (effects (font (size 1.27 1.27)) (justify right bottom))
   )
-  (text "ESP32 Stepper Motor Analyzer 1.4.0" (at 183.515 175.26 0)
+  (text "ESP32 Stepper Motor Analyzer 1.4.1" (at 183.515 175.26 0)
     (effects (font (size 2 2)) (justify left bottom))
   )
@@
     (pin "1")
   )
-  (symbol (lib_id "power:+3V3") (at 147.955 37.465 270) (unit 1)
-    (in_bom yes) (on_board yes)
-    (property "Reference" "#PWR0108" (id 0) (at 144.145 37.465 0)
-      (effects (font (size 1.27 1.27)) hide)
-    )
-    (property "Value" "+3V3" (id 1) (at 149.225 35.56 90))
-    (property "Footprint" "" (id 2) (at 147.955 37.465 0)
-      (effects (font (size 1.27 1.27)) hide)
-    )
-    (property "Datasheet" "" (id 3) (at 147.955 37.465 0)
+  (symbol (lib_id "power:+3V3") (at 149.225 37.465 270) (unit 1)
+    (in_bom yes) (on_board yes)
+    (property "Reference" "#PWR0108" (id 0) (at 145.415 37.465 0)
+      (effects (font (size 1.27 1.27)) hide)
+    )
+    (property "Value" "+3V3" (id 1) (at 150.495 35.56 90))
+    (property "Footprint" "" (id 2) (at 149.225 37.465 0)
+      (effects (font (size 1.27 1.27)) hide)
+    )
+    (property "Datasheet" "" (id 3) (at 149.225 37.465 0)
       (effects (font (size 1.27 1.27)) hide)
     )
@@
     (pin "2")
   )
-  (symbol (lib_id "Jumper:SolderJumper_2_Open") (at 138.43 37.465 0) (unit 1)
-    (in_bom no) (on_board yes) (fields_autoplaced)
-    (property "Reference" "JP1" (id 0) (at 138.43 35.4132 0))
-    (property "Value" "SolderJumper_2_Open" (id 1) (at 138.43 35.4131 0)
-      (effects (font (size 1.27 1.27)) hide)
-    )
-    (property "Footprint" "stepper_monitor:SolderJumper-2_P1.3mm_Open_RoundedPad1.0x1.5mm" (id 2) (at 138.43 37.465 0)
-      (effects (font (size 1.27 1.27)) hide)
-    )
-    (property "Datasheet" "~" (id 3) (at 138.43 37.465 0)
-      (effects (font (size 1.27 1.27)) hide)
-    )
-    (pin "1")
-    (pin "2")
-  )
   (symbol (lib_id "Device:C_Small") (at 261.62 123.825 180) (unit 1)
     (in_bom yes) (on_board yes)
@@
     (pin "2")
   )
+  (symbol (lib_id "Device:R_Small_US") (at 139.7 37.465 270) (unit 1)
+    (in_bom yes) (on_board yes)
+    (property "Reference" "R19" (id 0) (at 141.605 35.56 90))
+    (property "Value" "0R" (id 1) (at 137.16 35.56 90))
+    (property "Footprint" "Resistor_SMD:R_0402_1005Metric" (id 2) (at 139.7 37.465 0)
+      (effects (font (size 1.27 1.27)) hide)
+    )
+    (property "Datasheet" "~" (id 3) (at 139.7 37.465 0)
+      (effects (font (size 1.27 1.27)) hide)
+    )
+    (property "LCSC" "C17168" (id 4) (at 140.335 40.005 90))
+    (pin "1")
+    (pin "2")
+  )
   (symbol (lib_id "stepper_monitor:DC_DC") (at 82.55 37.465 0) (unit 1)
     (in_bom yes) (on_board yes)
@@
     (pin "2")
   )
-  (symbol (lib_id "power:PWR_FLAG") (at 144.145 36.83 0) (unit 1)
-    (in_bom yes) (on_board yes)
-    (property "Reference" "#FLG0102" (id 0) (at 144.145 34.925 0)
-      (effects (font (size 1.27 1.27)) hide)
-    )
-    (property "Value" "PWR_FLAG" (id 1) (at 144.145 32.385 0))
-    (property "Footprint" "" (id 2) (at 144.145 36.83 0)
-      (effects (font (size 1.27 1.27)) hide)
-    )
-    (property "Datasheet" "~" (id 3) (at 144.145 36.83 0)
+  (symbol (lib_id "power:PWR_FLAG") (at 145.415 36.83 0) (unit 1)
+    (in_bom yes) (on_board yes)
+    (property "Reference" "#FLG0102" (id 0) (at 145.415 34.925 0)
+      (effects (font (size 1.27 1.27)) hide)
+    )
+    (property "Value" "PWR_FLAG" (id 1) (at 145.415 32.385 0))
+    (property "Footprint" "" (id 2) (at 145.415 36.83 0)
+      (effects (font (size 1.27 1.27)) hide)
+    )
+    (property "Datasheet" "~" (id 3) (at 145.415 36.83 0)
       (effects (font (size 1.27 1.27)) hide)
     )
@@
       (reference "J5") (unit 1) (value "JTAG") (footprint "stepper_monitor:PinHeader_2x05_P1.27mm_Vertical_SMD")
     )
-    (path "/9d03fff4-c295-4428-baee-9254e712f3b4"
-      (reference "JP1") (unit 1) (value "SolderJumper_2_Open") (footprint "stepper_monitor:SolderJumper-2_P1.3mm_Open_RoundedPad1.0x1.5mm")
-    )
     (path "/64c584ec-f1bc-453f-8b60-7c99d996b567"
       (reference "M1") (unit 1) (value "Motor-simple_stepper_motor_analyzer") (footprint "stepper_monitor:Empty")
@@
       (reference "R18") (unit 1) (value "5K1") (footprint "Resistor_SMD:R_0402_1005Metric")
     )
+    (path "/c2470c78-9c3a-433f-a1eb-b1a3e5c72178"
+      (reference "R19") (unit 1) (value "0R") (footprint "Resistor_SMD:R_0402_1005Metric")
+    )
     (path "/b7f5be08-e26a-42d3-899d-e4457a8f22ac"

Commit message: Simplify the power supply using a diode based design.
Parts:
- removed D5: 5V6, stepper_monitor:D_MiniMELF_zenner, symbol stepper_monitor:zenner
- removed Q2: PJA3439, stepper_monitor:SOT-23, symbol stepper_monitor:P_MOSFET
- removed R12: 300K, Resistor_SMD:R_0402_1005Metric, symbol Device:R_Small_US
- removed R13: 20K, Resistor_SMD:R_0402_1005Metric, symbol Device:R_Small_US
- added C3: 100n, Capacitor_SMD:C_0402_1005Metric, symbol Device:C_Small
- added D3: SM4007PL, stepper_monitor:D2_SOD-123, symbol Diode:1N4005
- added D6: B5819W, stepper_monitor:D_SOD-123, symbol Device:D_Schottky
- added R3: 200K, Resistor_SMD:R_0402_1005Metric, symbol Device:R_Small_US
- added R8, R9: 10K, Resistor_SMD:R_0402_1005Metric, symbol Device:R_Small_US
- D5: renamed from D4; value D_Schottky -> B5819W
- JJ5: renamed from J5; LCSC C2935458 -> DNP
- renumbered C2 to C1, C3 to C10, C4 to C11, C16 to C12, C15 to C13, C11 to C14, C12 to C15, C17 to C16, C13 to C17, C14 to C18, C18 to C19, C8 to C2, C5 to C4, C9 to C5, C10 to C6, C6 to C7, C1 to C8, C7 to C9, D3 to D4, R4 to R1, R11 to R10, R18 to R11, R7 to R12, R10 to R13, R8 to R14, R9 to R15, R19 to R16, R16 to R17, R17 to R18, R14 to R19, R5 to R2, R15 to R20, R1 to R4, R2 to R5, R3 to R6, R6 to R7, U4 to U1, U1 to U2, U2 to U3, U5 to U4, U6 to U5, U3 to U6
Connections:
- net GNDD: now also C3.1, R3.2, R8.1, R9.1
- net VBUS: now also R9.2
- net at C6.2, C8.2, D5.1 (K)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: now also D6.1 (K); no longer C5.2, U1.3 (OUT)
- net at C1.2, C2.2, U1.1 (IN): now also D3.1 (K), R3.1
- net at J3.2 (Pin_2): now also D3.2 (A)
- new net: C3.2, C5.2, D6.2 (A), R8.2, U1.3 (OUT)
Other:
- note added: "CC6920BSO-5A"
- note added: "R17"
- note added: "R18"
- note added: "Reserved 1"
- note added: "Reserved 2"
- note added: "Solder LCSC C2935458 For JTAG Debugging"
- note added: "TMCS1108A4B"
- note added: "X"
- moved on the sheet: C1, C10, C11, C2, C5, C6, C8, D5, J3, R16, R17, R18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
