File: hardware/stepper_monitor.kicad_pcb (KiCad board)
At the start: 2 copper layers, 38.5 x 43 mm, 58 parts, among them J1 Conn_01x04_Male, J2 Conn_01x04_Male, J3 Conn_01x02_Male, J4 USB_C_Receptacle_USB2.0, Q1 MMDT2222A, SW1 SW_Push, U1 5V, U2 CP2102N-A01-GQFN28, U3 AMS1117-3.3, U4 CC6920BSO-5A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

Commit message: Renamed jj5 to j5. Increased version to 1.4.2. This is one commit past order of 1.4.1 from JLCPCB.
Parts:
- renumbered JJ5 to J5
Other:
- board text added: "V1.4.2"
- board text removed: "V1.4.1"
Changed lines of the file:
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@@
   (net 5 "Net-(C18-Pad2)")
   (net 6 "Net-(D4-Pad2)")
-  (net 7 "unconnected-(JJ5-Pad1)")
-  (net 8 "unconnected-(JJ5-Pad10)")
+  (net 7 "unconnected-(J5-Pad1)")
+  (net 8 "unconnected-(J5-Pad10)")
   (net 9 "Net-(R7-Pad1)")
   (net 10 "GNDD")
@@
     (property "Sheetname" "")
     (attr smd)
-    (fp_text reference "JJ5" (at -4.235 0 90) (layer "F.SilkS") hide
+    (fp_text reference "J5" (at -4.235 0 90) (layer "F.SilkS") hide
       (effects (font (size 1 1) (thickness 0.15)))
     )
@@
     (fp_line (start 1.07 1.705) (end 1.07 2.75) (layer "F.Fab") (width 0.1))
     (pad "1" smd rect (at -2.54 1.95 180) (size 0.74 2.4) (layers "F.Cu" "F.Paste" "F.Mask")
-      (net 7 "unconnected-(JJ5-Pad1)") (pinfunction "Pin_1") (pintype "passive+no_connect"))
+      (net 7 "unconnected-(J5-Pad1)") (pinfunction "Pin_1") (pintype "passive+no_connect"))
     (pad "2" smd rect (at -2.54 -1.95 180) (size 0.74 2.4) (layers "F.Cu" "F.Paste" "F.Mask")
       (net 58 "ESP_TMS") (pinfunction "Pin_2") (pintype "passive"))
@@
       (net 10 "GNDD") (pinfunction "Pin_9") (pintype "passive"))
     (pad "10" smd rect (at 2.54 -1.95 180) (size 0.74 2.4) (layers "F.Cu" "F.Paste" "F.Mask")
-      (net 8 "unconnected-(JJ5-Pad10)") (pinfunction "Pin_10") (pintype "passive+no_connect"))
+      (net 8 "unconnected-(J5-Pad10)") (pinfunction "Pin_10") (pintype "passive+no_connect"))
     (model "${KISYS3DMOD}/Connector_PinHeader_1.27mm.3dshapes/PinHeader_2x05_P1.27mm_Vertical_SMD.wrl"
       (offset (xyz 0 0 0))
@@
     (effects (font (size 1.27 1.27) (thickness 0.2032)))
   )
-  (gr_text "V1.4.1" (at 17.1958 -23.8252 90) (layer "F.SilkS")
+  (gr_text "V1.4.2" (at 17.1958 -23.8252 90) (layer "F.SilkS")
     (effects (font (size 1.2 1.2) (thickness 0.3)) (justify left))
   )

Commit message: Upgraded kicad to 7.0 (design version incremented to 1.4.2)
Parts:
- J1, J2: value Conn_01x04_Male -> Conn_01x04_Pin
- J3: value Conn_01x02_Male -> Conn_01x02_Pin
Other:
- board text added: "V 1.4.2"
- board text removed: "V1.4.2"
